Commit message: Add monitor package and robot motion functionalities
- Created setup.cfg and setup.py for the monitor package.
- Added copyright and flake8 tests for code quality assurance.
- Updated RViz configuration to include a target point marker.
- Enhanced gazebo launch file to include a new node for robot motion.
- Updated package.xml to include dependencies for robot_motion.
- Modified URDF to adjust robot base orientation and joint limits.
- Updated SDF world file to correctly position the robot in the workcell.
- Added robot motion package with homogenous transformations, inverse kinematics, and velocity profile calculations.
- Implemented a turnNode for controlling robot joint movements with visualization of trajectory.
- Added utility functions for matrix operations and trajectory generation.

File: src/my_robot_description/urdf/robot.urdf (robot description, URDF)
Before this commit: robot my_robot_description, 8 links, 7 joints
Joints:
- joint Joint5: limit lower=-2.0 upper=2.0 effort=100 velocity=1 -> lower=-2.35619449 upper=2.35619449 effort=100 velocity=1
- joint world_to_base: origin xyz=0 0 0 rpy=0 0 0 -> xyz=0 0 0 rpy=0 0 3.141592654

Commit message: Add robot kinematics package and integrate joint monitoring
- Introduced `robot_kinematics` package for shared kinematics, including forward/inverse kinematics and joint conventions.
- Updated `my_robot_description` launch files to include `joint_monitor` node for real-time joint state monitoring.
- Modified URDF joint limits for improved accuracy.
- Adjusted Gazebo world file to disable gravity for simulation.
- Enhanced `robot_motion` package to utilize new kinematics functionalities and joint conventions.
- Added comprehensive README documentation for `robot_kinematics` detailing usage, configuration, and monitoring.
- Implemented joint conventions management to ensure consistent feedback and command conversions.
- Created tests for joint conventions to validate functionality and error handling.

File: src/my_robot_description/urdf/robot.urdf (robot description, URDF)
Before this commit: robot my_robot_description, 8 links, 7 joints
Joints:
- joint Joint2: limit lower=-1.1345 upper=2.0944 effort=100 velocity=1 -> lower=-1.25 upper=2.24 effort=100 velocity=1
- joint Joint3: limit lower=-3.14 upper=1.28 effort=100 velocity=1 -> lower=-3.88 upper=1.45 effort=100 velocity=1
- joint Joint5: limit lower=-2.35619449 upper=2.35619449 effort=100 velocity=1 -> lower=-2.26 upper=2.26 effort=100 velocity=1
